Commit message: Added 6th joint and fixed upper meshes

File: rbx1_urdf/urdf/rbx1.urdf (robot description, URDF)
Before this commit: robot rbx1_urdf, 12 links, 11 joints
Links:
- removed link Gripper_Idol_Gear
- removed link Gripper_Servo_Gear
- removed link Link_1
- removed link Link_2
- removed link Link_3
- removed link Link_4
- removed link Link_5
- removed link Pivot_Arm_Gripper_Idol
- removed link Pivot_Arm_Gripper_Servo
- removed link Tip_Gripper_Idol
- removed link Tip_Gripper_Servo
- added link gripper_idol_gear, mass 0.0051273; collision mesh filename=package://rbx1_urdf/meshes/gripper_idol_gear.STL; visual mesh filename=package://rbx1_urdf/meshes/gripper_idol_gear.STL
- added link gripper_servo_gear, mass 0.0048997; collision mesh filename=package://rbx1_urdf/meshes/gripper_servo_gear.STL; visual mesh filename=package://rbx1_urdf/meshes/gripper_servo_gear.STL
- added link link_1_shoulder, mass 4.2526; collision mesh filename=package://rbx1_urdf/meshes/link_1_shoulder.STL; visual mesh filename=package://rbx1_urdf/meshes/link_1_shoulder.STL
- added link link_2_arm, mass 1.9323; collision mesh filename=package://rbx1_urdf/meshes/link_2_arm.STL; visual mesh filename=package://rbx1_urdf/meshes/link_2_arm.STL
- added link link_3_upper_forearm, mass 1.1381; collision mesh filename=package://rbx1_urdf/meshes/link_3_upper_forearm.STL; visual mesh filename=package://rbx1_urdf/meshes/link_3_upper_forearm.STL
- added link link_4_forearm, mass 0.62964; collision mesh filename=package://rbx1_urdf/meshes/link_4_forearm.STL; visual mesh filename=package://rbx1_urdf/meshes/link_4_forearm.STL
- added link link_5_wrist, mass 0.15; collision mesh filename=package://rbx1_urdf/meshes/link_5_wrist.STL; visual mesh filename=package://rbx1_urdf/meshes/link_5_wrist.STL
- added link link_6_hand, mass 0.04; collision mesh filename=package://rbx1_urdf/meshes/link_6_hand.STL; visual mesh filename=package://rbx1_urdf/meshes/link_6_hand.STL
- added link pivot_arm_gripper_idol, mass 0.0018597; collision mesh filename=package://rbx1_urdf/meshes/pivot_arm_gripper_idol.STL; visual mesh filename=package://rbx1_urdf/meshes/pivot_arm_gripper_idol.STL
- added link pivot_arm_gripper_servo, mass 0.0018597; collision mesh filename=package://rbx1_urdf/meshes/pivot_arm_gripper_servo.STL; visual mesh filename=package://rbx1_urdf/meshes/pivot_arm_gripper_servo.STL
- added link tip_gripper_idol, mass 0.010676; collision mesh filename=package://rbx1_urdf/meshes/tip_gripper_idol.STL; visual mesh filename=package://rbx1_urdf/meshes/tip_gripper_idol.STL
- added link tip_gripper_servo, mass 0.010676; collision mesh filename=package://rbx1_urdf/meshes/tip_gripper_servo.STL; visual mesh filename=package://rbx1_urdf/meshes/tip_gripper_servo.STL
Joints:
- removed joint Gripper_Idol_Gear_Joint
- removed joint Gripper_Servo_Gear_Joint
- removed joint Joint_1
- removed joint Joint_2
- removed joint Joint_3
- removed joint Joint_4
- removed joint Joint_5
- removed joint Pivot_Arm_Gripper_Idol_Joint
- removed joint Pivot_Arm_Gripper_Servo_Joint
- removed joint Tip_Gripper_Idol_Joint
- removed joint Tip_Gripper_Servo_Joint
- added joint gripper_idol_gear_joint: type revolute, parent link_6_hand, child gripper_idol_gear, origin xyz=-0.024233 -0.013715 -0.00052 rpy=1.5708 0.0 1.5708, axis 0 1 0, limit lower=0 upper=-1.5707 effort=5 velocity=1
- added joint gripper_servo_gear_joint: type revolute, parent link_6_hand, child gripper_servo_gear, origin xyz=-0.024077 0.014019 0.003057 rpy=1.5708 0.0 -1.5708, axis 0 1 0, limit lower=0 upper=1.5707 effort=5 velocity=1
- added joint joint_1_base_shoulder: type revolute, parent base_link, child link_1_shoulder, origin xyz=0 -0.2425 0 rpy=1.5708 9.5417E-17 2.7766, axis 0 1 0, limit lower=-1 upper=1 effort=5 velocity=1
- added joint joint_2_shoulder_arm: type revolute, parent link_1_shoulder, child link_2_arm, origin xyz=0 0.18264 0 rpy=-3.1416 0.95134 1.5708, axis 0 -1 0, limit lower=-1 upper=1 effort=5 velocity=1
- added joint joint_3_arm_upper_forearm: type revolute, parent link_2_arm, child link_3_upper_forearm, origin xyz=0 0 -0.22112 rpy=-3.1416 0.98126 -3.1416, axis 0 -1 0, limit lower=-1 upper=1 effort=5 velocity=1
- added joint joint_4_upper_forearm_forearm: type revolute, parent link_3_upper_forearm, child link_4_forearm, origin xyz=0.16988 -0.00099213 0 rpy=3.1416 -1.2279 1.5708, axis 0.010353 -0.99993 -0.0059382, limit lower=-1 upper=1 effort=5 velocity=1
- added joint joint_5_forearm_wrist: type revolute, parent link_4_forearm, child link_5_wrist, origin xyz=-0.0021346 0.053041 0.0016936 rpy=-1.5639 -0.091135 -0.00062919, axis 0 1 0, limit lower=-1 upper=1 effort=5 velocity=1
- added joint joint_6_wrist_hand: type revolute, parent link_5_wrist, child link_6_hand, origin xyz=-0.034 0.0 0.024 rpy=0 0.645772 0, axis 1 0 0, limit lower=-1 upper=1 effort=5 velocity=1
- added joint pivot_arm_gripper_idol_joint: type revolute, parent link_6_hand, child pivot_arm_gripper_idol, origin xyz=-0.044291 -0.007028 -0.000002 rpy=1.5708 0.0 -1.5708, axis 0 1 0, limit lower=-1 upper=1 effort=5 velocity=1, mimic joint=gripper_idol_gear_joint multiplier=1 offset=0
- added joint pivot_arm_gripper_servo_joint: type revolute, parent link_6_hand, child pivot_arm_gripper_servo, origin xyz=-0.044253 0.007042 -0.000282 rpy=1.5708 0.0 -1.6308, axis 0 1 0, limit lower=-1 upper=1 effort=5 velocity=1, mimic joint=gripper_servo_gear_joint multiplier=1 offset=0
- added joint tip_gripper_idol_joint: type revolute, parent gripper_idol_gear, child tip_gripper_idol, origin xyz=-0.040206 0 -0.001701 rpy=-3.1416 0.5236 -3.1416, axis 0 1 0, limit lower=-1 upper=1 effort=5 velocity=1, mimic joint=gripper_idol_gear_joint multiplier=-1 offset=0
- added joint tip_gripper_servo_joint: type revolute, parent gripper_servo_gear, child tip_gripper_servo, origin xyz=-0.039906 -0.004 -0.0027473 rpy=-3.1416 -1.5569 -2.0392E-12, axis 0 1 0, limit lower=0 upper=1.3 effort=5 velocity=1, mimic joint=gripper_servo_gear_joint multiplier=1 offset=0

Commit message: Simplified collision meshes

File: rbx1_urdf/urdf/rbx1.urdf (robot description, URDF)
Before this commit: robot rbx1_urdf, 13 links, 12 joints
Links:
- added link world
- link gripper_idol_gear: geometry collision mesh filename=package://rbx1_urdf/meshes/collision/gripper_idol_gear.STL; visual mesh filename=package://rbx1_urdf/meshes/gripper_idol_gear.STL
- link gripper_servo_gear: geometry collision mesh filename=package://rbx1_urdf/meshes/collision/gripper_servo_gear.STL; visual mesh filename=package://rbx1_urdf/meshes/gripper_servo_gear.STL
- link link_1_shoulder: geometry collision mesh filename=package://rbx1_urdf/meshes/collision/link_1_shoulder.STL; visual mesh filename=package://rbx1_urdf/meshes/link_1_shoulder.STL
- link link_2_arm: geometry collision mesh filename=package://rbx1_urdf/meshes/collision/link_2_arm.STL; visual mesh filename=package://rbx1_urdf/meshes/link_2_arm.STL
- link link_3_upper_forearm: geometry collision mesh filename=package://rbx1_urdf/meshes/collision/link_3_upper_forearm.S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; visual mesh filename=package://rbx1_urdf/meshes/link_3_upper_forearm.STL
- link link_4_forearm: geometry collision mesh filename=package://rbx1_urdf/meshes/collision/link_4_forearm.STL; visual mesh filename=package://rbx1_urdf/meshes/link_4_forearm.STL
- link link_5_wrist: geometry collision mesh filename=package://rbx1_urdf/meshes/collision/link_5_wrist.STL; visual mesh filename=package://rbx1_urdf/meshes/link_5_wrist.STL
- link link_6_hand: geometry collision mesh filename=package://rbx1_urdf/meshes/collision/link_6_hand.STL; visual mesh filename=package://rbx1_urdf/meshes/link_6_hand.STL
- link pivot_arm_gripper_idol: geometry collision mesh filename=package://rbx1_urdf/meshes/collision/pivot_arm_gripper_idol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; visual mesh filename=package://rbx1_urdf/meshes/pivot_arm_gripper_idol.STL
- link pivot_arm_gripper_servo: geometry collision mesh filename=package://rbx1_urdf/meshes/collision/pivot_arm_gripper_serv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; visual mesh filename=package://rbx1_urdf/meshes/pivot_arm_gripper_servo.STL
- link tip_gripper_idol: geometry collision mesh filename=package://rbx1_urdf/meshes/collision/tip_gripper_idol.STL; visual mesh filename=package://rbx1_urdf/meshes/tip_gripper_idol.STL
- link tip_gripper_servo: geometry collision mesh filename=package://rbx1_urdf/meshes/collision/tip_gripper_servo.STL; visual mesh filename=package://rbx1_urdf/meshes/tip_gripper_servo.STL
Joints:
- added joint fixed: type fixed, parent world, child base_link

Commit message: Simplified inertia of gripper to avoid physics getting wacky

File: rbx1_urdf/urdf/rbx1.urdf (robot description, URDF)
Before this commit: robot rbx1_urdf, 14 links, 13 joints
Links:
- link base_link: geometry collision mesh filename=package://rbx1_urdf/meshes/collision/base_link.STL; visual mesh filename=package://rbx1_urdf/meshes/base_link.STL

Commit message: Joint simulator ROS controllers

File: rbx1_urdf/urdf/rbx1.urdf (robot description, URDF)
Before this commit: robot rbx1_urdf, 14 links, 13 joints
Joints:
- joint gripper_idol_gear_joint: limit lower=0 upper=-1.5707 effort=5 velocity=1 -> lower=0 upper=1.5707 effort=5 velocity=1; origin xyz=-0.024233 -0.013715 -0.00052 rpy=1.5708 0.0 1.5708 -> xyz=-0.024233 -0.013715 -0.00052 rpy=4.71239 0.0 1.5708
- joint pivot_arm_gripper_idol_joint: origin xyz=-0.044291 -0.007028 -0.000002 rpy=1.5708 0.0 -1.5708 -> xyz=-0.044291 -0.007028 -0.000002 rpy=4.71239 0.0 -1.5708
- joint tip_gripper_idol_joint: limit lower=-1 upper=1 effort=5 velocity=1 -> lower=0 upper=1.3 effort=5 velocity=1; origin xyz=-0.040206 0 -0.001701 rpy=-3.1416 0.5236 -3.1416 -> xyz=-0.040206 0 -0.001701 rpy=0.0 -0.5236 -3.1416

Commit message: upright default pose and file server to transfer urdf to unity

File: rbx1_urdf/urdf/rbx1.urdf (robot description, URDF)
Before this commit: robot rbx1_urdf, 14 links, 13 joints
Joints:
- joint joint_1_base_shoulder: origin xyz=0 -0.2425 0 rpy=1.5708 9.5417E-17 2.7766 -> xyz=0 -0.2425 0 rpy=1.5708 9.5417E-17 0
- joint joint_2_shoulder_arm: origin xyz=0 0.18264 0 rpy=-3.1416 0.95134 1.5708 -> xyz=0 0.18264 0 rpy=-3.1416 1.5708 1.5708
- joint joint_3_arm_upper_forearm: origin xyz=0 0 -0.22112 rpy=-3.1416 0.98126 -3.1416 -> xyz=0 0 -0.22112 rpy=-3.1416 1.5708 -3.1416
- joint joint_4_upper_forearm_forearm: origin xyz=0.16988 -0.00099213 0 rpy=3.1416 -1.2279 1.5708 -> xyz=0.16988 -0.00099213 0 rpy=3.1416 1.5708   1.5708
- joint joint_5_forearm_wrist: origin xyz=-0.0021346 0.053041 0.0016936 rpy=-1.5639 -0.091135 -0.00062919 -> xyz=-0.0021346 0.053041 0.0016936 rpy=-1.5639 -0.091135 -1.0472

Commit message: Modifies limit of robot og urdf and pos based on radians

File: rbx1_urdf/urdf/rbx1.urdf (robot description, URDF)
Before this commit: robot rbx1_urdf, 14 links, 13 joints
Joints:
- joint joint_1_base_shoulder: limit lower=-1 upper=1 effort=5 velocity=1 -> lower=-1.5707975 upper=1.07993 effort=5 velocity=1
- joint joint_2_shoulder_arm: limit lower=-1 upper=1 effort=5 velocity=1 -> lower=-1.5707975 upper=1.5707975 effort=5 velocity=1
- joint joint_3_arm_upper_forearm: limit lower=-1 upper=1 effort=5 velocity=1 -> lower=-1.9635 upper=1.9635 effort=5 velocity=1
- joint joint_4_upper_forearm_forearm: limit lower=-1 upper=1 effort=5 velocity=1 -> lower=-3.141595 upper=3.141595 effort=5 velocity=1
- joint joint_5_forearm_wrist: limit lower=-1 upper=1 effort=5 velocity=1 -> lower=-1.7952 upper=1.7951 effort=5 velocity=1
- joint joint_6_wrist_hand: limit lower=-1 upper=1 effort=5 velocity=1 -> lower=-3.141595 upper=3.141595 effort=5 velocity=1

Commit message: Camera sensor in gazebo

File: rbx1_urdf/urdf/rbx1.urdf (robot description, URDF)
Before this commit: robot rbx1_urdf, 14 links, 13 joints
Links:
- added link camera_link, mass 0.010676; collision box size=0.05 0.05 0.05; visual box size=0.05 0.05 0.05
Joints:
- added joint camera_joint: type fixed, parent base_link, child camera_link, origin xyz=0.6 0.6 0.5 rpy=0 0 -1.95, axis 0 1 0

Commit message: Gripper node

File: rbx1_urdf/urdf/rbx1.urdf (robot description, URDF)
Before this commit: robot rbx1_urdf, 15 links, 14 joints
Joints:
- joint pivot_arm_gripper_idol_joint: limit lower=-1 upper=1 effort=5 velocity=1 -> lower=-1.5 upper=0 effort=5 velocity=1
- joint tip_gripper_idol_joint: limit lower=0 upper=1.3 effort=5 velocity=1 -> lower=0 upper=1.4 effort=5 velocity=1
